File: rack_frontpanel_leds.kicad_pcb (KiCad board)
At the start: 2 copper layers, 33 x 24.5 mm, 24 parts, among them P1 CONN_2X2, P2 CONN_2X2, P3 CONN_2X2, P4 CONN_2X2

Commit message: added through-hole LEDs in parallel with red on RGB-LED 1..3
Parts:
- added D10: LED, LEDs:LED-3MM, B.Cu at (76.4, 75.9)
- added D11: LED, LEDs:LED-3MM, B.Cu at (85.2, 75.9)
- added D9: LED, LEDs:LED-3MM, B.Cu at (67.6, 75.9)
Routing:
- net Net-(D11-Pad2): track 16.7 -> 25.4 mm
- net Net-(D10-Pad2): track 26.0 -> 34.6 mm
- net Net-(D1-Pad1): track 34.9 -> 43.5 mm
- net Net-(D12-Pad2): track 36.4 -> 43.3 mm
- net Net-(D11-Pad1): track 22.3 -> 27.7 mm
- net Net-(D1-Pad4): track 20.0 -> 25.2 mm
- net Net-(D10-Pad1): track 17.7 -> 22.8 mm
- net Net-(D12-Pad1): track 31.9 -> 30.4 mm
