File: rack_frontpanel_leds.sch (KiCad schematic (older format))
At the start: 20 parts, among them P1 CONN_2X2, P2 CONN_2X2, P3 CONN_2X2, P4 CONN_2X2

Commit message: added through-hole LEDs in parallel with red on RGB-LED 1..3
Parts:
- added D10, D11, D9: LED, symbol LED
Connections:
- net at D1.4 (A), D2.4 (A), P1.1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: now also D9.1 (A)
- net at D1.1 (KR), D2.1 (KR), P1.2: now also D9.2 (K)
- net at D3.4 (A), D4.4 (A), P2.1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: now also D10.1 (A)
- net at D3.1 (KR), D4.1 (KR), P2.2: now also D10.2 (K)
- net at D5.4 (A), D6.4 (A), P3.1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: now also D11.1 (A)
- net at D5.1 (KR), D6.1 (KR), P3.2: now also D11.2 (K)
Changed lines of the file:
@@
 Connection ~ 8650 1100
 Wire Wire Line
+	7400 1100 7800 1100
+$Comp
+L LED D9
+U 1 1 54CF08FD
+P 1300 2500
+F 0 "D9" H 1300 2600 50  0000 C CNN
+F 1 "LED" H 1300 2400 50  0000 C CNN
+F 2 "" H 1300 2500 60  0000 C CNN
+F 3 "" H 1300 2500 60  0000 C CNN
+	1    1300 2500
+	-1   0    0    1
+$EndComp
+$Comp
+L LED D10
+U 1 1 54CF0AF7
+P 3450 2500
+F 0 "D10" H 3450 2600 50  0000 C CNN
+F 1 "LED" H 3450 2400 50  0000 C CNN
+F 2 "" H 3450 2500 60  0000 C CNN
+F 3 "" H 3450 2500 60  0000 C CNN
+	1    3450 2500
+	-1   0    0    1
+$EndComp
+$Comp
+L LED D11
+U 1 1 54CF0BE4
+P 5600 2500
+F 0 "D11" H 5600 2600 50  0000 C CNN
+F 1 "LED" H 5600 2400 50  0000 C CNN
+F 2 "" H 5600 2500 60  0000 C CNN
+F 3 "" H 5600 2500 60  0000 C CNN
+	1    5600 2500
+	-1   0    0    1
+$EndComp
+Wire Wire Line
+	5900 1950 5900 2500
+Wire Wire Line
+	5900 2500 5800 2500
+Wire Wire Line
+	5400 2500 5200 2500
+Wire Wire Line
+	5200 2500 5200 1750
+Wire Wire Line
+	5200 1750 5350 1750
+Wire Wire Line
+	3750 1950 3750 2500
+Wire Wire Line
+	3750 2500 3650 2500
+Wire Wire Line
+	3250 2500 3050 2500
+Wire Wire Line
+	3050 2500 3050 1750
+Wire Wire Line
+	3050 1750 3200 1750
+Wire Wire Line
+	1600 1950 1600 2500
+Wire Wire Line
+	1600 2500 1500 2500
+Wire Wire Line
+	1100 2500 900  2500
+Wire Wire Line
+	900  2500 900  1750
+Wire Wire Line
+	900  1750 1050 1750
+Wire Wire Line
 	7400 2150 7400 1100
-Wire Wire Line
-	7400 1100 7800 1100
 $EndSCHEMATC
